File: sch&pcb/IRProxy.sch (KiCad schematic (older format))
At the start: 34 parts, among them IC1 ASM1117 33, IC2 PIC16F18313-I/P, J1 BARREL_JACK, J2 BARREL_JACK, J3 CONN_01X04_MALE, M1 ESP-12E, Q1 BSS98, Q2 2N3906, Q3 2N3906

Commit message: Se unifica la dependencia en IRProxy.lib
Se adapta el esquemático para eliminar los archivos *rescue y *cache, en este punto las partes incluidas en el solo dependen de IRProxy.lib
Parts:
- C1, C2, C3: symbol CP1_Small -> Device:CP1_Small
- C4, C5: symbol C_Small -> Device:C_Small
- D1: symbol D_Small -> Device:D_Small
- D2: symbol D_Shockley -> Device:D_Shockley
- DZ: symbol D_Zener -> Device:D_Zener
- IC1: symbol LD1117S33CTR -> IRProxy:LD1117S33CTR
- IC2: symbol PIC16F18313-I/P -> IRProxy:PIC16F18313-I_P
- J1, J2: symbol BARREL_JACK -> IRProxy:conn_BARREL_JACK
- J3: symbol CONN_01X04_MALE -> IRProxy:conn_CONN_01X04_MALE
- JP1: symbol Jumper_NO_Small -> Device:Jumper_NO_Small
- L1: symbol L_Core_Ferrite -> Device:L_Core_Ferrite
- LD1, LD2, LD3: symbol LED_ALT -> Device:LED_ALT
- M1: symbol ESP-12E-RESCUE-IRProxy -> IRProxy:ESP-12E
- Q1: symbol Q_NMOS_DGS -> Device:Q_NMOS_DGS
- Q2: symbol Q_PNP_EBC -> Device:Q_PNP_EBC
- Q3: symbol Q_NPN_EBC -> Device:Q_NPN_EBC
- R1, R10, R11, R12, R13, R2, R3, R4, R5, R7, R8, R9: symbol R -> Device:R
Connections:
- wire segments 100 -> 139
Changed lines of the file:
@@
-EESchema Schematic File Version 2
-LIBS:IRProxy-rescue
-LIBS:power
-LIBS:device
-LIBS:transistors
-LIBS:conn
-LIBS:linear
-LIBS:regul
-LIBS:74xx
-LIBS:cmos4000
-LIBS:adc-dac
-LIBS:memory
-LIBS:xilinx
-LIBS:microcontrollers
-LIBS:dsp
-LIBS:microchip
-LIBS:analog_switches
-LIBS:motorola
-LIBS:texas
-LIBS:intel
-LIBS:audio
-LIBS:interface
-LIBS:digital-audio
-LIBS:philips
-LIBS:display
-LIBS:cypress
-LIBS:siliconi
-LIBS:opto
-LIBS:atmel
-LIBS:contrib
-LIBS:valves
-LIBS:microchip_dspic33dsc
-LIBS:microchip_pic10mcu
-LIBS:microchip_pic12mcu
-LIBS:microchip_pic16mcu
-LIBS:microchip_pic18mcu
-LIBS:microchip_pic24mcu
-LIBS:microchip_pic32mcu
-LIBS:estandares
-LIBS:Symbols_DCDC-ACDC-Converter_RevC_20Jul2012
-LIBS:Symbols_Socket-DIN41612_RevA
-LIBS:ESP8266
-LIBS:IRProxy-cache
-EELAYER 25 0
+EESchema Schematic File Version 4
+EELAYER 29 0
 EELAYER END
 $Descr A4 11693 8268
@@
 $EndDescr
 $Comp
-L BARREL_JACK J1
+L IRProxy:conn_BARREL_JACK J1
 U 1 1 590BEFE2
 P 1100 1600
@@
 $EndComp
 $Comp
-L BARREL_JACK J2
+L IRProxy:conn_BARREL_JACK J2
 U 1 1 590BF035
 P 1100 3650
@@
 $EndComp
 $Comp
-L D_Small D1
+L Device:D_Small D1
 U 1 1 590BF04E
 P 1800 1500
@@
 $EndComp
 $Comp
-L D_Shockley D2
+L Device:D_Shockley D2
 U 1 1 590BF0C4
 P 2400 2250
@@
 $EndComp
 $Comp
-L Q_NMOS_DGS Q1
+L Device:Q_NMOS_DGS Q1
 U 1 1 590BF10D
 P 2500 3250
@@
 $EndComp
 $Comp
-L CP1_Small C1
+L Device:CP1_Small C1
 U 1 1 590BF177
 P 2000 2700
@@
 $EndComp
 $Comp
-L CP1_Small C2
+L Device:CP1_Small C2
 U 1 1 590BF1B8
 P 2900 2250
@@
 $EndComp
 $Comp
-L LD1117S33CTR IC1
+L IRProxy:LD1117S33CTR IC1
 U 1 1 590BF1E7
 P 3800 1550
@@
 $EndComp
 $Comp
-L L_Core_Ferrite L1
+L Device:L_Core_Ferrite L1
 U 1 1 590BF224
 P 2650 2750
@@
 $EndComp
 $Comp
-L R R2
+L Device:R R2
 U 1 1 590BFA5A
 P 3050 3500
@@
 $EndComp
 $Comp
-L R R3
+L Device:R R3
 U 1 1 590C0063
 P 5450 1800
@@
 $EndComp
 $Comp
-L LED_ALT LD1
+L Device:LED_ALT LD1
 U 1 1 590C08D4
 P 5700 3400
@@
 $EndComp
 $Comp
-L R R4
+L Device:R R4
 U 1 1 590C09F9
 P 5700 3000
@@
 $EndComp
 $Comp
-L PIC16F18313-I/P IC2
+L IRProxy:PIC16F18313-I_P IC2
 U 1 1 590C13D1
 P 8300 1650
@@
 $EndComp
 $Comp
-L GND #PWR01
+L power:GND #PWR01
 U 1 1 590C1414
 P 4300 5250
@@
 $EndComp
 $Comp
-L ESP-12E-RESCUE-IRProxy M1
+L IRProxy:ESP-12E M1
 U 1 1 590C19D6
 P 7950 4050
@@
 $EndComp
 $Comp
-L Q_NPN_EBC Q3
+L Device:Q_NPN_EBC Q3
 U 1 1 590C2354
 P 5800 2500
@@
 $EndComp
 $Comp
-L R R5
+L Device:R R5
 U 1 1 590C2483
 P 6050 2200
@@
 $EndComp
 $Comp
-L R R10
+L Device:R R10
 U 1 1 590C2586
 P 9200 3300
@@
 $EndComp
 $Comp
-L LED_ALT LD2
+L Device:LED_ALT LD2
 U 1 1 590C25F9
 P 9200 2900
@@
 $EndComp
 $Comp
-L R R11
+L Device:R R11
 U 1 1 590C2778
 P 9500 3300
@@
 $EndComp
 $Comp
-L LED_ALT LD3
+L Device:LED_ALT LD3
 U 1 1 590C277E
 P 9500 2900
@@
 $EndComp
 $Comp
-L R R9
+L Device:R R9
 U 1 1 590C2B92
 P 9150 4800
@@
 $EndComp
 $Comp
-L R R8
+L Device:R R8
 U 1 1 590C2EF9
 P 8950 3300
@@
 $EndComp
 $Comp
-L R R12
+L Device:R R12
 U 1 1 590C31BF
 P 9750 3300
@@
 $EndComp
 $Comp
-L R R7
+L Device:R R7
 U 1 1 590C3407
 P 6400 4850
@@
 $EndComp
 $Comp
-L Jumper_NO_Small JP1
+L Device:Jumper_NO_Small JP1
 U 1 1 590C3B15
 P 9750 4450
@@
 $EndComp
 $Comp
-L CONN_01X04_MALE J3
+L IRProxy:conn_CONN_01X04_MALE J3
 U 1 1 590C3E46
 P 10250 3800
@@
 GND
 $Comp
-L CP1_Small C3
+L Device:CP1_Small C3
 U 1 1 590C8153
 P 4300 2275
@@
 $EndComp
 $Comp
-L R R1
+L Device:R R1
 U 1 1 590C8671
 P 2200 3300
@@
 NoConn ~ 7900 4950
 $Comp
-L C_Small C4
+L Device:C_Small C4
 U 1 1 590D2ECE
 P 4650 2250
@@
 $EndComp
 Wire Wire Line
-	1400 1500 1700 1500
+	1400 1500 1600 1500
 Wire Wire Line
 	1600 1500 1600 3550
@@
 	1500 1700 1500 3750
 Wire Wire Line
-	1400 3750 3050 3750
+	1400 3750 1500 3750
 Wire Wire Line
 	2000 3750 2000 2800
@@
 Connection ~ 1600 1500
 Wire Wire Line
-	1900 1500 3400 1500
+	1900 1500 2000 1500
 Wire Wire Line
 	2000 1500 2000 2600
@@
 Connection ~ 2000 1500
 Wire Wire Line
-	2400 2400 2400 3050
+	2400 2400 2400 2750
 Wire Wire Line
 	2400 3750 2400 3450
@@
 	3050 3250 3050 3350
 Wire Wire Line
-	2200 2750 2500 2750
+	2200 2750 2400 2750
 Connection ~ 2400 2750
 Wire Wire Line
-	2800 2750 4650 2750
+	2800 2750 2900 2750
 Wire Wire Line
 	2900 2750 2900 2350
@@
 	3800 1800 3800 2750
 Wire Wire Line
-	4300 2375 4300 5250
+	4300 2375 4300 2750
 Connection ~ 2900 2750
 Wire Wire Line
 	4950 3250 4950 2000
 Wire Wire Line
-	2700 3250 4950 3250
+	2700 3250 3050 3250
 Connection ~ 3050 3250
 Wire Wire Line
 	4950 1500 4950 1600
 Wire Wire Line
-	4200 1500 6500 1500
+	4200 1500 4300 1500
 Wire Wire Line
 	5700 5200 5700 3550
@@
 	6250 4450 7050 4450
 Wire Wire Line
-	6250 1500 6250 4450
-Wire Wire Line
-	6250 2600 9950 2600
+	6250 1500 6250 2600
+Wire Wire Line
+	6250 2600 8950 2600
 Connection ~ 4300 5200
 Wire Wire Line
@@
 Connection ~ 9500 2600
 Wire Wire Line
-	9750 3450 9750 4350
+	9750 3450 9750 4150
 Wire Wire Line
 	9750 4150 8850 4150
@@
 	6400 3950 7050 3950
 Wire Wire Line
-	6400 1800 6400 4700
+	6400 1800 6400 2850
 NoConn ~ 6500 1950
 $Comp
-L Q_PNP_EBC Q2
+L Device:Q_PNP_EBC Q2
 U 1 1 590BFF80
 P 5050 1800
@@
 	5300 1800 5250 1800
 Wire Wire Line
-	10750 5200 4300 5200
+	10750 5200 9950 5200
 Wire Wire Line
 	6500 1650 5875 1650
@@
 Connection ~ 6400 5200
 $Comp
-L C_Small C5
+L Device:C_Small C5
 U 1 1 5914CD22
 P 6600 4850
@@
 $EndComp
 Wire Wire Line
-	6600 3500 6600 4750
+	6600 3500 6600 3750
 Wire Wire Line
 	6600 4950 6600 5200
 Connection ~ 6600 5200
 $Comp
-L R R13
+L Device:R R13
 U 1 1 5914D137
 P 6600 3350
@@
 Su huella no aparece\nen el PCB.
 $Comp
-L D_Zener DZ
+L Device:D_Zener DZ
 U 1 1 5C808DFD
 P 3325 2250
@@
 	0    1    1    0
 $EndComp
+Wire Wire Line
+	1500 3750 2000 3750
+Wire Wire Line
+	1600 1500 1700 1500
+Wire Wire Line
+	2000 1500 2400 1500
+Wire Wire Line
+	2000 3750 2200 3750
+Wire Wire Line
+	2400 3750 3050 3750
+Wire Wire Line
+	2400 2750 2400 3050
+Wire Wire Line
+	2400 2750 2500 2750
+Wire Wire Line
+	2400 1500 2900 1500
+Wire Wire Line
+	2900 1500 3325 1500
+Wire Wire Line
+	2900 2750 3325 2750
+Wire Wire Line
+	3050 3250 4950 3250
+Wire Wire Line
+	3800 2750 4300 2750
+Wire Wire Line
+	4950 1500 6250 1500
+Wire Wire Line
+	6250 1500 6500 1500
+Wire Wire Line
+	4300 5200 4300 5250
+Wire Wire Line
+	6250 2600 6250 4450
+Wire Wire Line
+	9200 2600 9500 2600
+Wire Wire Line
+	8950 5200 7000 5200
+Wire Wire Line
+	9150 5200 8950 5200
+Wire Wire Line
+	8950 2600 9200 2600
+Wire Wire Line
+	9500 2600 9750 2600
+Wire Wire Line
+	9950 5200 9750 5200
+Wire Wire Line
+	9750 4150 9750 4350
+Wire Wire Line
+	9750 5200 9150 5200
+Wire Wire Line
+	4300 1500 4650 1500
+Wire Wire Line
+	4300 2750 4300 5200
+Wire Wire Line
+	4300 2750 4650 2750
+Wire Wire Line
+	2200 3750 2400 3750
+Wire Wire Line
+	4650 1500 4950 1500
+Wire Wire Line
+	9750 2600 9950 2600
+Wire Wire Line
+	5700 5200 4300 5200
+Wire Wire Line
+	6400 3950 6400 4700
+Wire Wire Line
+	6400 5200 5700 5200
+Wire Wire Line
+	6600 5200 6400 5200
+Wire Wire Line
+	6600 3750 6600 4750
+Wire Wire Line
+	6400 2850 6400 3950
+Wire Wire Line
+	7000 5200 6600 5200
+Wire Wire Line
+	3325 2750 3800 2750
+Wire Wire Line
+	3325 1500 3400 1500
 $EndSCHEMATC
